File: Modules/Flashlight/PCB/LED/LED.kicad_pcb (KiCad board)
At the start: 2 copper layers, 74 x 21.5 mm, 36 parts

Commit message: Added everything
Parts:
- added REF**: MountingHole_2.2mm_M2, MountingHole:MountingHole_2.2mm_M2, B.Cu at (109.7, 82.0)
- added REF**: MountingHole_2.2mm_M2, MountingHole:MountingHole_2.2mm_M2, B.Cu at (178.7, 98.5)
- moved REF** 70.9 mm to (178.7, 82.0), turned to 0 degrees
- moved REF** 70.8 mm to (109.7, 98.5), turned to 0 degrees
- moved TP1 0.60 mm to (112.2, 88.3)
- moved TP2 0.30 mm to (112.2, 92.5)
Other:
- board text removed: "Pikne"
