File: Modules/LiPo charger/PCB/LiPo charger Rev 1.0.kicad_pcb (KiCad board)
At the start: 2 copper layers, 72 x 26.7 mm, 117 parts, among them IC1 ISOM8111DFGR, IC2 TPS55288RPMR, IC3 ISOM8111DFGR, IC4 ISOM8111DFGR, J1 Battery, J2 Conn_01x05_Socket, J3 UP32-1-C-H-G-BMT-P24, J4 FFC2B35-06-G, J5 UART, J6 Conn_01x04_Socket, Q1 AO3400A, Q10 DMP3014SFDE-13, Q2 AO3400A, Q3 NTTFS5C454NLTAG, Q4 NTTFS5C454NLTAG, Q5 AO3400A, Q6 AO3400A, Q7 DMP3014SFDE-13, Q8 DMP3014SFDE-13, Q9 AO3400A, SW1 SW_Push, U1 TVS2200DRV, U2 STUSB4500QTR, U3 ER_OLEDM0.91_1x-I2C, U4 STM32L011G3Ux, U5 TPS562246DRLR

Commit message: Added everything
Parts:
- turned C14 to 180 degrees
Routing:
- net GND: vias 59 -> 63
Changed lines of the file:
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@@
 	(footprint "Capacitor_SMD:C_1206_3216Metric"
 		(layer "F.Cu")
-		(at 111.025 75.75)
+		(at 111.025 75.75 180)
 		(descr "Capacitor SMD 1206 (3216 Metric), square (rectangular) end terminal, IPC-7351 nominal, (Body size source: IPC-SM-782 page 76, https://www.pcb-3d.com/wordpress/wp-content/uploads/ipc-sm-782a_amendment_1_and_2.pdf)")
 		(tags "capacitor")
 		(property "Reference" "C14"
-			(at 3.675 -0.45 0)
+			(at -3.675 0.55 0)
 			(layer "F.SilkS")
 			(effects
@@
 		(duplicate_pad_numbers_are_jumpers no)
 		(fp_line
-			(start -0.711252 -0.91)
-			(end 0.711252 -0.91)
+			(start -0.711252 0.91)
+			(end 0.711252 0.91)
 			(stroke
 				(width 0.12)
@@
 		)
 		(fp_line
-			(start -0.711252 0.91)
-			(end 0.711252 0.91)
+			(start -0.711252 -0.91)
+			(end 0.711252 -0.91)
 			(stroke
 				(width 0.12)
@@
 		)
 		(pad "1" smd roundrect
-			(at -1.475 0)
+			(at -1.475 0 180)
 			(size 1.15 1.8)
 			(layers "F.Cu" "F.Mask" "F.Paste")
@@
 		)
 		(pad "2" smd roundrect
-			(at 1.475 0)
+			(at 1.475 0 180)
 			(size 1.15 1.8)
 			(layers "F.Cu" "F.Mask" "F.Paste")
@@
 	)
 	(via
+		(at 136.507 76.4)
+		(size 0.7)
+		(drill 0.4)
+		(layers "F.Cu" "B.Cu")
+		(free yes)
+		(net "GND")
+	)
+	(via
 		(at 137.68 90.8)
 		(size 0.7)
@@
 	)
 	(via
+		(at 135.7 76.4)
+		(size 0.7)
+		(drill 0.4)
+		(layers "F.Cu" "B.Cu")
+		(free yes)
+		(net "GND")
+	)
+	(via
 		(at 107.6 78.75)
 		(size 0.7)
@@
 	)
 	(via
+		(at 136.534 77.3)
+		(size 0.7)
+		(drill 0.4)
+		(layers "F.Cu" "B.Cu")
+		(free yes)
+		(net "GND")
+	)
+	(via
 		(at 108.5 75.435)
 		(size 0.7)
@@
 	)
 	(via
+		(at 135.707 77.3)
+		(size 0.7)
+		(drill 0.4)
+		(layers "F.Cu" "B.Cu")
+		(free yes)
+		(net "GND")
+	)
+	(via
 		(at 137.707 91.7)
 		(size 0.7)
@@
 	)
 	(segment
-		(start 152.214587 90.114587)
-		(end 151.9 89.8)
+		(start 152.233801 90.362758)
+		(end 152.214587 90.381972)
 		(width 0.2)
 		(layer "B.Cu")
@@
 	)
 	(segment
-		(start 143.6 89.8)
-		(end 142.25 91.15)
+		(start 151.9 89.8)
+		(end 143.6 89.8)
 		(width 0.2)
 		(layer "B.Cu")
@@
 	)
 	(segment
-		(start 142.25 91.15)
-		(end 142.25 91.74)
+		(start 143.6 89.8)
+		(end 142.25 91.15)
 		(width 0.2)
 		(layer "B.Cu")
@@
 	)
 	(segment
-		(start 152.233801 90.362758)
-		(end 152.214587 90.381972)
+		(start 142.25 91.15)
+		(end 142.25 91.74)
 		(width 0.2)
 		(layer "B.Cu")
@@
 	)
 	(segment
-		(start 151.9 89.8)
-		(end 143.6 89.8)
+		(start 152.214587 90.114587)
+		(end 151.9 89.8)
 		(width 0.2)
 		(layer "B.Cu")
@@
 	)
 	(zone
+		(layer "B.Cu")
+		(hatch edge 0.5)
+		(connect_pads
+			(clearance 0)
+		)
+		(min_thickness 0.25)
+		(keepout
+			(tracks allowed)
+			(vias allowed)
+			(pads allowed)
+			(copperpour not_allowed)
+			(footprints allowed)
+		)
+		(placement
+			(enabled no)
+			(sheetname "")
+		)
+		(fill
+			(thermal_gap 0.5)
+			(thermal_bridge_width 0.5)
+			(island_removal_mode 0)
+		)
+		(polygon
+			(pts
+				(xy 144.2 90.6) (xy 145.5 90.6) (xy 145.5 91) (xy 144.2 91)
+			)
+		)
+	)
+	(zone
 		(net "+3.3V")
 		(layer "B.Cu")
@@
 		(polygon
 			(pts
-				(xy 146 93.6) (xy 146 91.4) (xy 146.5 89.835) (xy 146.5 87.8) (xy 144.144444 87.8) (xy 141 87.5)
+				(xy 146 93.6) (xy 145.996582 92.398587) (xy 145.5 92.4) (xy 145.5 87.8) (xy 144.144444 87.8) (xy 141 87.5)
 				(xy 140 92.4) (xy 140 93.6)
 			)
