File: BMS/BMS Rev 1.1.kicad_sch (KiCad schematic)
At the start: 34 parts, among them IC1 BQ41Z50RSNR, J2 out, J3 out, J4 in, J5 in, Q1 CSD18502Q5B, Q2 CSD18502Q5B

Commit message: Added BOMs and updated some PCB files
Parts:
- removed D1: LED, LED_SMD:LED_0402_1005Metric_Pad0.77x0.64mm_HandSolder, symbol Device:LED
- removed JP1, JP2, JP3, JP4: SolderJumper_2_Open, Jumper:SolderJumper-2_P1.3mm_Open_RoundedPad1.0x1.5mm, symbol Jumper:SolderJumper_2_Open
- removed NT2: NetTie_2, NetTie:NetTie-2_SMD_Pad0.5mm, symbol Device:NetTie_2
- removed R5: 3m, Resistor_SMD:R_2512_6332Metric_Pad1.40x3.35mm_HandSolder, symbol Device:R
- added C8: 1nf, Capacitor_SMD:C_0402_1005Metric, symbol Device:C
- added R5: 3m, Resistor_SMD:R_Shunt_Vishay_WSK2512_6332Metric_T2.21mm, symbol Device:R_Shunt
- added SW1: WAKE, Button_Switch_SMD:SW_SPST_B3U-1000P, symbol Switch:SW_Push
- added SW2: SHUTDN, Button_Switch_SMD:SW_SPST_B3U-1000P, symbol Switch:SW_Push
- C1, C2, C3, C4, C6, C7: footprint Capacitor_SMD:C_0402_1005Metric_Pad0.74x0.62mm_HandSolder -> Capacitor_SMD:C_0402_1005Metric
- C5: footprint Capacitor_SMD:C_0201_0603Metric_Pad0.64x0.40mm_HandSolder -> Capacitor_SMD:C_0402_1005Metric
- Q1, Q2: value CSD18502Q5B -> CSD18512Q5B
- R1, R6: footprint Resistor_SMD:R_0603_1608Metric_Pad0.98x0.95mm_HandSolder -> Resistor_SMD:R_0603_1608Metric
- R10, R11, R12, R2, R3, R4, R7, R8, R9: footprint Resistor_SMD:R_0402_1005Metric_Pad0.72x0.64mm_HandSolder -> Resistor_SMD:R_0402_1005Metric
- R13: value 220 -> 10k; footprint Resistor_SMD:R_0402_1005Metric_Pad0.72x0.64mm_HandSolder -> Resistor_SMD:R_0603_1608Metric
Connections:
- net B+: now also R13.1, R4.2; no longer R1.2, R3.2
- net B+ out: now also R1.2, SW1.2
- net B- out: now also R5.4; no longer R10.2
- net CELL1: now also R3.2; no longer R4.2
- net GND: now also J4.3 (Pin_3), J4.4 (Pin_4), R2.2, C8.1, R5.1, SW2.1
- net at C3.2, IC1.21 (VC2), R4.1: now also IC1.19 (VC4), IC1.20 (VC3)
- net at R13.2: now also SW1.1; no longer IC1.6 (GPIO3)
- net at IC1.7 (~{PRES}/_~{SHUTDN}): now also C8.2, SW2.2
- removed net GNDPWR: J4.3 (Pin_3), J4.4 (Pin_4), R11.2, R2.2
- new net: R11.2, R5.2
- new net: R10.2, R5.3
- no-connect marks 10 -> 8
Other:
- title: (none) -> Pikne BMS
- moved on the sheet: C5, J2, J3, J4, J5, R1, R10, R11
