File: Main PCB/Pikne Rev 1.1.kicad_sch (KiCad schematic)
At the start: 110 parts, among them J1 USB_C_Receptacle_PowerOnly_6P, J2 bat, J3 Conn_01x03_Pin, J4 i2c, J6 program, SW1 SW_Push, SW2 SW_Push, U1 BQ25792RQMR, U2 ATmega328P-A, U3 OLED 0.91 inch, U4 PTPS25751DREFR, U5 TVS2200DRV, U6 TPS54531DDAR, U7 TLV75533PDBV, U8 CAT24C256, U9 TPS259461ARPW

Commit message: Added BOMs and updated some PCB files
Parts:
- added R26: 4.7k, Resistor_SMD:R_0603_1608Metric, symbol Device:R
- C36: footprint Capacitor_SMD:C_0402_1005Metric_Pad0.74x0.62mm_HandSolder -> Capacitor_SMD:C_0603_1608Metric
- L3: footprint SPM6550:SPM6550 -> Inductor:7443845030010
Connections:
- net +3V3: now also R26.1
- net alert: now also R26.2
Changed lines of the file:
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@@
 	(wire
 		(pts
+			(xy 375.92 33.02) (xy 375.92 31.75)
+		)
+		(stroke
+			(width 0)
+			(type default)
+		)
+	)
+	(wire
+		(pts
 			(xy 347.98 31.75) (xy 347.98 34.29)
 		)
@@
 		)
 	)
+	(label "alert"
+		(at 375.92 33.02 0)
+		(effects
+			(font
+				(size 1.27 1.27)
+			)
+			(justify left bottom)
+		)
+	)
 	(label "SDRV"
 		(at 137.16 85.09 0)
@@
 	)
 	(symbol
+		(lib_id "power:+3V3")
+		(at 375.92 24.13 0)
+		(unit 1)
+		(body_style 1)
+		(exclude_from_sim no)
+		(in_bom yes)
+		(on_board yes)
+		(in_pos_files yes)
+		(dnp no)
+		(fields_autoplaced yes)
+		(property "Reference" "#PWR073"
+			(at 375.92 27.94 0)
+			(hide yes)
+			(show_name no)
+			(do_not_autoplace no)
+			(effects
+				(font
+					(size 1.27 1.27)
+				)
+			)
+		)
+		(property "Value" "+3V3"
+			(at 375.92 19.05 0)
+			(show_name no)
+			(do_not_autoplace no)
+			(effects
+				(font
+					(size 1.27 1.27)
+				)
+			)
+		)
+		(property "Footprint" ""
+			(at 375.92 24.13 0)
+			(hide yes)
+			(show_name no)
+			(do_not_autoplace no)
+			(effects
+				(font
+					(size 1.27 1.27)
+				)
+			)
+		)
+		(property "Datasheet" ""
+			(at 375.92 24.13 0)
+			(hide yes)
+			(show_name no)
+			(do_not_autoplace no)
+			(effects
+				(font
+					(size 1.27 1.27)
+				)
+			)
+		)
+		(property "Description" "Power symbol creates a global label with name \"+3V3\""
+			(at 375.92 24.13 0)
+			(hide yes)
+			(show_name no)
+			(do_not_autoplace no)
+			(effects
+				(font
+					(size 1.27 1.27)
+				)
+			)
+		)
+		(pin "1"
+		)
+		(instances
+			(project "Pikne Rev 1.1"
+				(path "/0a0d1d9c-f6cd-4de5-98f3-3ca6235ec442"
+					(reference "#PWR073")
+					(unit 1)
+				)
+			)
+		)
+	)
+	(symbol
 		(lib_id "Device:C")
 		(at 293.37 46.99 0)
@@
 			)
 		)
-		(property "Footprint" "Capacitor_SMD:C_0402_1005Metric_Pad0.74x0.62mm_HandSolder"
+		(property "Footprint" "Capacitor_SMD:C_0603_1608Metric"
 			(at 156.5148 146.05 0)
 			(hide yes)
@@
 	)
 	(symbol
+		(lib_id "Device:R")
+		(at 375.92 27.94 0)
+		(unit 1)
+		(body_style 1)
+		(exclude_from_sim no)
+		(in_bom yes)
+		(on_board yes)
+		(in_pos_files yes)
+		(dnp no)
+		(property "Reference" "R26"
+			(at 374.142 29.21 0)
+			(show_name no)
+			(do_not_autoplace no)
+			(effects
+				(font
+					(size 1.27 1.27)
+				)
+				(justify right)
+			)
+		)
+		(property "Value" "4.7k"
+			(at 374.142 26.67 0)
+			(show_name no)
+			(do_not_autoplace no)
+			(effects
+				(font
+					(size 1.27 1.27)
+				)
+				(justify right)
+			)
+		)
+		(property "Footprint" "Resistor_SMD:R_0603_1608Metric"
+			(at 374.142 27.94 90)
+			(hide yes)
+			(show_name no)
+			(do_not_autoplace no)
+			(effects
+				(font
+					(size 1.27 1.27)
+				)
+			)
+		)
+		(property "Datasheet" ""
+			(at 375.92 27.94 0)
+			(hide yes)
+			(show_name no)
+			(do_not_autoplace no)
+			(effects
+				(font
+					(size 1.27 1.27)
+				)
+			)
+		)
+		(property "Description" "Resistor"
+			(at 375.92 27.94 0)
+			(hide yes)
+			(show_name no)
+			(do_not_autoplace no)
+			(effects
+				(font
+					(size 1.27 1.27)
+				)
+			)
+		)
+		(pin "1"
+		)
+		(pin "2"
+		)
+		(instances
+			(project "Pikne Rev 1.1"
+				(path "/0a0d1d9c-f6cd-4de5-98f3-3ca6235ec442"
+					(reference "R26")
+					(unit 1)
+				)
+			)
+		)
+	)
+	(symbol
 		(lib_id "power:-BATT")
 		(at 201.93 97.79 180)
@@
 			)
 		)
-		(property "Footprint" "SPM6550:SPM6550"
+		(property "Footprint" "Inductor:7443845030010"
 			(at 259.842 104.648 0)
 			(show_name no)
